Commit message: fixes turning right problem

File: src/TutorialF1tenth/urdf/macros.xacro (robot description, xacro)
@@ -10,5 +10,5 @@
 </xacro:macro>
 <xacro:macro name="left_wheels_inertial_params">
-  <origin xyz="0 0 -0.0225" rpy="0 0 0" />
+  <origin xyz="0 0 0" rpy="0 0 0" />
   <mass value="0.34055" />
   <inertia ixx="0.00026046" ixy="0"          ixz="0"
@@ -17,5 +17,5 @@
 </xacro:macro>
 <xacro:macro name="right_wheels_inertial_params">
-  <origin xyz="0 0 0.0225" rpy="0 0 0" />
+  <origin xyz="0 0 0" rpy="0 0 0" />
   <mass value="0.34055" />
   <inertia ixx="0.00026046" ixy="0"          ixz="0"
@@ -81,5 +81,5 @@
 </xacro:macro>
 <xacro:macro name="left_wheels_collision_geometry">
-  <origin xyz="0 0 -0.0225" rpy="0 0 0" />
+  <origin xyz="0 0 0" rpy="0 0 0" />
   <geometry>
     <cylinder length="0.045" radius="0.05" />
@@ -87,5 +87,5 @@
 </xacro:macro>
 <xacro:macro name="right_wheels_collision_geometry">
-  <origin xyz="0 0 0.0225" rpy="0 0 0" />
+  <origin xyz="0 0 0" rpy="0 0 0" />
   <geometry>
     <cylinder length="0.045" radius="0.05" />

File: src/TutorialF1tenth/urdf/racecar.xacro (robot description, xacro)
@@ -77,10 +77,10 @@
     </visual>
   </link>
-  <joint name="left_steering_hinge_joint" type="revolute">
-    <origin xyz="0.325 0.1 0" rpy="0 1.5708 0" />
-    <parent link="chassis" />
-    <child link="left_steering_hinge" />
-    <axis xyz="-1 0 0" />
-    <limit lower="-1.0" upper="1.0" effort="10" velocity="100" />
+  <joint name="left_steering_hinge_joint" type="continuous">
+       <origin xyz="0.325 0.1 0" rpy="0 0 0" />  <!-- Removed the 90° Y rotation -->
+       <parent link="chassis" />
+       <child link="left_steering_hinge" />
+       <axis xyz="0 0 1" />  <!-- Now rotates around Z-axis (vertical) -->
+       <limit lower="-1.0" upper="1.0" effort="10" velocity="100" />
   </joint>
   <xacro:steering_hinge_transmission name="left_steering_hinge" />
@@ -96,9 +96,9 @@
   </link>
   <joint name="right_steering_hinge_joint" type="continuous">
-    <origin xyz="0.325 -0.1 0" rpy="0 1.5708 0" />
-    <parent link="chassis" />
-    <child link="right_steering_hinge" />
-    <axis xyz="-1 0 0" />
-    <limit lower="-1.0" upper="1.0" effort="10" velocity="100" />
+       <origin xyz="0.325 -0.1 0" rpy="0 0 0" />  <!-- Removed the 90° Y rotation -->
+       <parent link="chassis" />
+       <child link="right_steering_hinge" />
+       <axis xyz="0 0 1" />  <!-- Now rotates around Z-axis (vertical) -->
+       <limit lower="-1.0" upper="1.0" effort="10" velocity="100" />
   </joint>
   <xacro:steering_hinge_transmission name="right_steering_hinge" />
@@ -116,5 +116,5 @@
     </collision>
   </link>
-  <joint name="left_front_wheel_joint" type="fixed">
+  <joint name="left_front_wheel_joint" type="continuous">
     <origin xyz="0 0 0" rpy="1.5708 0 0" />
     <parent link="left_steering_hinge" />
@@ -136,5 +136,5 @@
     </collision>
   </link>
-  <joint name="right_front_wheel_joint" type="fixed">
+  <joint name="right_front_wheel_joint" type="continuous">
     <origin xyz="0 0 0" rpy="1.5708 0 0" />
     <parent link="right_steering_hinge" />
